Commit message: Updated URDF with rubber tires

File: redox_robot_description/urdf/redox_robot.xacro (robot description, xacro)
@@ -26,7 +26,7 @@
 <link name="wheel_3">
   <inertial>
-    <origin xyz="0.02664362537853835 -5.397499067000266e-07 1.4559471091246667e-07" rpy="0 0 0"/>
-    <mass value="3.1717827199849116"/>
-    <inertia ixx="0.008134" iyy="0.00516" izz="0.00516" ixy="0.0" iyz="0.0" ixz="0.0"/>
+    <origin xyz="0.02729659083369923 -0.0003579998502422632 -0.00014058126175340354" rpy="0 0 0"/>
+    <mass value="4.750258601717646"/>
+    <inertia ixx="0.014935" iyy="0.009074" izz="0.009066" ixy="2e-06" iyz="4e-06" ixz="1e-06"/>
   </inertial>
   <visual>
@@ -46,7 +46,7 @@
 <link name="wheel_2">
   <inertial>
-    <origin xyz="-0.026643352957820027 -2.287799444750105e-07 1.4559471170003113e-07" rpy="0 0 0"/>
-    <mass value="3.1717827199849116"/>
-    <inertia ixx="0.008134" iyy="0.00516" izz="0.00516" ixy="0.0" iyz="-0.0" ixz="-0.0"/>
+    <origin xyz="-0.027296318412980913 0.0003572313203910604 -0.00014058126175261598" rpy="0 0 0"/>
+    <mass value="4.750258601717646"/>
+    <inertia ixx="0.014935" iyy="0.009074" izz="0.009066" ixy="2e-06" iyz="-4e-06" ixz="-1e-06"/>
   </inertial>
   <visual>
@@ -66,7 +66,7 @@
 <link name="wheel_4">
   <inertial>
-    <origin xyz="0.026643625378538316 -5.397499067555378e-07 1.4559471092460974e-07" rpy="0 0 0"/>
-    <mass value="3.1717827199849116"/>
-    <inertia ixx="0.008134" iyy="0.00516" izz="0.00516" ixy="0.0" iyz="0.0" ixz="0.0"/>
+    <origin xyz="0.027296590833699196 -0.00035799985024231873 -0.00014058126175339226" rpy="0 0 0"/>
+    <mass value="4.750258601717646"/>
+    <inertia ixx="0.014935" iyy="0.009074" izz="0.009066" ixy="2e-06" iyz="4e-06" ixz="1e-06"/>
   </inertial>
   <visual>
@@ -86,7 +86,7 @@
 <link name="wheel_1">
   <inertial>
-    <origin xyz="-0.026643352957819957 -2.287799444750105e-07 1.4559471170176586e-07" rpy="0 0 0"/>
-    <mass value="3.1717827199849116"/>
-    <inertia ixx="0.008134" iyy="0.00516" izz="0.00516" ixy="0.0" iyz="-0.0" ixz="-0.0"/>
+    <origin xyz="-0.027296318412980844 0.0003572313203910882 -0.0001405812617526125" rpy="0 0 0"/>
+    <mass value="4.750258601717646"/>
+    <inertia ixx="0.014935" iyy="0.009074" izz="0.009066" ixy="2e-06" iyz="-4e-06" ixz="-1e-06"/>
   </inertial>
   <visual>
