Commit message: Update URDF + catkin.sh

File: ros package/redox_robot_description/urdf/redox_robot.xacro (robot description, xacro)
@@ -553,3 +553,10 @@
   <child link="thermal_camera_1"/>
 </joint>
+<link name="world" />
+  <joint name="orientation" type="fixed">
+    <origin xyz="0 0 0" rpy="3.14159265359 0 1.57079632679" />
+    <parent link="world" />
+    <child link="base_link" />
+  </joint>
+</link>
 </robot>

Commit message: World frame

File: ros package/redox_robot_description/urdf/redox_robot.xacro (robot description, xacro)
@@ -559,4 +559,3 @@
     <child link="base_link" />
   </joint>
-</link>
 </robot>
